File: Hardware/DinoCalcPCB/DinoCalcPCB.brd (EAGLE design)
At the start: 100 x 80 mm, 6 parts, among them U1 ATMEGA328P_PDIP

Commit message: update
Parts:
- added C1: 0.1uF, SparkFun-Capacitors:CAP-PTH-SMALL
- added J1: AVR_SPI, SparkFun-Connectors:2X3_OFFSET
- added R1: 10K, SparkFun-Resistors:AXIAL-0.4
- added S1: (no value), SparkFun-Electromechanical:TACTILE-PTH
- JP1: value (none) -> BATTERY
- JP3: value (none) -> KEYPAD
Connections:
- new net GND: C1.2, J1.6, JP1.1, JP2.3, S1.1, U1.22, U1.8
- new net LED_GRN: JP2.1, U1.27
- new net LED_RED: JP2.2, U1.28
- new net N$1: JP3.1, U1.2
- new net N$10: J1.1, U1.18
- new net N$13: J1.5, R1.P$1, S1.3, U1.1
- new net N$14: J1.3, U1.19
- new net N$2: JP3.2, U1.3
- new net N$3: JP3.3, U1.4
- new net N$4: JP3.4, U1.5
- new net N$5: JP3.5, U1.6
- new net N$6: JP3.6, U1.11
- new net N$7: JP3.7, U1.12
- new net N$8: JP3.8, U1.13
- new net N$9: J1.4, U1.17
- new net VCC: C1.1, J1.2, JP1.2, R1.P$2, U1.20, U1.7
Changed lines of the file:
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@@
 <elements>
 <element name="U1" library="SparkFun-DigitalIC" package="DIL28-3" value="ATMEGA328P_PDIP" x="35.56" y="30.48" rot="R90"/>
-<element name="JP1" library="SparkFun-Connectors" package="1X02" value="" x="20.32" y="21.59"/>
+<element name="JP1" library="SparkFun-Connectors" package="1X02" value="BATTERY" x="20.32" y="21.59"/>
 <element name="JP2" library="SparkFun-Connectors" package="1X03" value="" x="8.89" y="13.97"/>
-<element name="JP3" library="SparkFun-Connectors" package="1X08" value="" x="49.53" y="13.97"/>
+<element name="JP3" library="SparkFun-Connectors" package="1X08" value="KEYPAD" x="49.53" y="13.97"/>
 <element name="LOGO1" library="SparkFun-Aesthetics" package="OSHW-LOGO-L" value="OSHW-LOGOL" x="8.89" y="6.35"/>
 <element name="FRAME1" library="SparkFun-Aesthetics" package="CREATIVE_COMMONS" value="FRAME-LETTER" x="21.59" y="-8.89"/>
+<element name="J1" library="SparkFun-Connectors" package="2X3_OFFSET" value="AVR_SPI" x="6.35" y="-15.24"/>
+<element name="C1" library="SparkFun-Capacitors" package="CAP-PTH-SMALL" value="0.1uF" x="1.27" y="-22.86"/>
+<element name="R1" library="SparkFun-Resistors" package="AXIAL-0.4" value="10K" x="6.35" y="-27.94"/>
+<element name="S1" library="SparkFun-Electromechanical" package="TACTILE-PTH" value="" x="8.89" y="30.48" rot="R180"/>
 </elements>
 <signals>
+<signal name="N$1">
+<contactref element="U1" pad="2"/>
+<contactref element="JP3" pad="1"/>
+<wire x1="39.37" y1="16.51" x2="49.53" y2="13.97" width="0" layer="19" extent="1-1"/>
+</signal>
+<signal name="N$2">
+<contactref element="JP3" pad="2"/>
+<contactref element="U1" pad="3"/>
+<wire x1="39.37" y1="19.05" x2="52.07" y2="13.97" width="0" layer="19" extent="1-1"/>
+</signal>
+<signal name="N$3">
+<contactref element="U1" pad="4"/>
+<contactref element="JP3" pad="3"/>
+<wire x1="39.37" y1="21.59" x2="54.61" y2="13.97" width="0" layer="19" extent="1-1"/>
+</signal>
+<signal name="N$4">
+<contactref element="JP3" pad="4"/>
+<contactref element="U1" pad="5"/>
+<wire x1="39.37" y1="24.13" x2="57.15" y2="13.97" width="0" layer="19" extent="1-1"/>
+</signal>
+<signal name="N$5">
+<contactref element="JP3" pad="5"/>
+<contactref element="U1" pad="6"/>
+<wire x1="39.37" y1="26.67" x2="59.69" y2="13.97" width="0" layer="19" extent="1-1"/>
+</signal>
+<signal name="N$7">
+<contactref element="U1" pad="12"/>
+<contactref element="JP3" pad="7"/>
+<wire x1="64.77" y1="13.97" x2="39.37" y2="41.91" width="0" layer="19" extent="1-1"/>
+</signal>
+<signal name="N$9">
+<contactref element="J1" pad="4"/>
+<contactref element="U1" pad="17"/>
+<wire x1="6.35" y1="-13.97" x2="31.75" y2="41.91" width="0" layer="19" extent="1-1"/>
+</signal>
+<signal name="N$10">
+<contactref element="J1" pad="1"/>
+<contactref element="U1" pad="18"/>
+<wire x1="3.81" y1="-16.51" x2="31.75" y2="39.37" width="0" layer="19" extent="1-1"/>
+</signal>
+<signal name="LED_GRN">
+<contactref element="JP2" pad="1"/>
+<contactref element="U1" pad="27"/>
+<wire x1="8.89" y1="13.97" x2="31.75" y2="16.51" width="0" layer="19" extent="1-1"/>
+</signal>
+<signal name="LED_RED">
+<contactref element="JP2" pad="2"/>
+<contactref element="U1" pad="28"/>
+<wire x1="11.43" y1="13.97" x2="31.75" y2="13.97" width="0" layer="19" extent="1-1"/>
+</signal>
+<signal name="GND">
+<contactref element="JP2" pad="3"/>
+<contactref element="J1" pad="6"/>
+<contactref element="JP1" pad="1"/>
+<contactref element="C1" pad="2"/>
+<contactref element="S1" pad="1"/>
+<contactref element="U1" pad="8"/>
+<contactref element="U1" pad="22"/>
+<wire x1="31.75" y1="29.21" x2="39.37" y2="31.75" width="0" layer="19" extent="1-1"/>
+<wire x1="20.32" y1="21.59" x2="31.75" y2="29.21" width="0" layer="19" extent="1-1"/>
+<wire x1="13.97" y1="13.97" x2="20.32" y2="21.59" width="0" layer="19" extent="1-1"/>
+<wire x1="12.1412" y1="28.2194" x2="20.32" y2="21.59" width="0" layer="19" extent="1-1"/>
+<wire x1="8.89" y1="-13.97" x2="13.97" y2="13.97" width="0" layer="19" extent="1-1"/>
+<wire x1="3.81" y1="-22.86" x2="8.89" y2="-13.97" width="0" layer="19" extent="1-1"/>
+</signal>
+<signal name="N$13">
+<contactref element="J1" pad="5"/>
+<contactref element="U1" pad="1"/>
+<contactref element="R1" pad="P$1"/>
+<contactref element="S1" pad="3"/>
+<wire x1="12.1412" y1="32.7406" x2="39.37" y2="13.97" width="0" layer="19" extent="1-1"/>
+<wire x1="8.89" y1="-16.51" x2="12.1412" y2="32.7406" width="0" layer="19" extent="1-1"/>
+<wire x1="1.27" y1="-27.94" x2="8.89" y2="-16.51" width="0" layer="19" extent="1-1"/>
+</signal>
+<signal name="N$6">
+<contactref element="JP3" pad="6"/>
+<contactref element="U1" pad="11"/>
+<wire x1="62.23" y1="13.97" x2="39.37" y2="39.37" width="0" layer="19" extent="1-1"/>
+</signal>
+<signal name="N$8">
+<contactref element="JP3" pad="8"/>
+<contactref element="U1" pad="13"/>
+<wire x1="67.31" y1="13.97" x2="39.37" y2="44.45" width="0" layer="19" extent="1-1"/>
+</signal>
+<signal name="N$14">
+<contactref element="U1" pad="19"/>
+<contactref element="J1" pad="3"/>
+<wire x1="6.35" y1="-16.51" x2="31.75" y2="36.83" width="0" layer="19" extent="1-1"/>
+</signal>
+<signal name="VCC">
+<contactref element="U1" pad="20"/>
+<contactref element="JP1" pad="2"/>
+<contactref element="C1" pad="1"/>
+<contactref element="U1" pad="7"/>
+<contactref element="J1" pad="2"/>
+<contactref element="R1" pad="P$2"/>
+<wire x1="31.75" y1="34.29" x2="39.37" y2="29.21" width="0" layer="19" extent="1-1"/>
+<wire x1="22.86" y1="21.59" x2="31.75" y2="34.29" width="0" layer="19" extent="1-1"/>
+<wire x1="3.81" y1="-13.97" x2="22.86" y2="21.59" width="0" layer="19" extent="1-1"/>
+<wire x1="1.27" y1="-22.86" x2="3.81" y2="-13.97" width="0" layer="19" extent="1-1"/>
+<wire x1="11.43" y1="-27.94" x2="1.27" y2="-22.86" width="0" layer="19" extent="1-1"/>
+</signal>
 </signals>
 </board>
